Commit message: Add per-joint friction and damping parameters

File: urdf/iiwa14.xacro (robot description, xacro)
@@ -10,8 +10,22 @@
   <xacro:property name="safety_controller_k_pos" value="100" />
   <xacro:property name="safety_controller_k_vel" value="2" />
-  <xacro:property name="joint_damping" value="0.5" />
-  <xacro:property name="joint_friction" value="1.0" />
   <xacro:property name="max_effort" value="300"/>
   <xacro:property name="max_velocity" value="10"/>
+   <xacro:property name="damping_factor" value="1.0"/>
+   <xacro:property name="d0" value="${damping_factor*0.1}"/>
+   <xacro:property name="d1" value="${damping_factor*0.1}"/>
+   <xacro:property name="d2" value="${damping_factor*0.1}"/>
+   <xacro:property name="d3" value="${damping_factor*0.1}"/>
+   <xacro:property name="d4" value="${damping_factor*0.1}"/>
+   <xacro:property name="d5" value="${damping_factor*0.1}"/>
+   <xacro:property name="d6" value="${damping_factor*0.1}"/>
+   <xacro:property name="friction_factor" value="1.0"/>
+   <xacro:property name="f0" value="${friction_factor*0.1}"/>
+   <xacro:property name="f1" value="${friction_factor*0.1}"/>
+   <xacro:property name="f2" value="${friction_factor*0.1}"/>
+   <xacro:property name="f3" value="${friction_factor*0.1}"/>
+   <xacro:property name="f4" value="${friction_factor*0.1}"/>
+   <xacro:property name="f5" value="${friction_factor*0.1}"/>
+   <xacro:property name="f6" value="${friction_factor*0.1}"/>
   <xacro:macro name="iiwa14" params="parent hardware_interface robot_name *origin">
     <!--joint between {parent} and link_0-->
@@ -60,5 +74,5 @@
            k_position="${safety_controller_k_pos}"
            k_velocity="${safety_controller_k_vel}"/>
-      <dynamics damping="${joint_damping}" friction="${joint_friction}"/>
+      <dynamics damping="${d0}" friction="${f0}"/>
     </joint>
     <link name="link_1">
@@ -95,5 +109,5 @@
            k_position="${safety_controller_k_pos}"
            k_velocity="${safety_controller_k_vel}"/>
-      <dynamics damping="${joint_damping}" friction="${joint_friction}"/>
+      <dynamics damping="${d1}" friction="${f1}"/>
     </joint>
     <link name="link_2">
@@ -130,5 +144,5 @@
            k_position="${safety_controller_k_pos}"
            k_velocity="${safety_controller_k_vel}"/>
-      <dynamics damping="${joint_damping}" friction="${joint_friction}"/>
+      <dynamics damping="${d2}" friction="${f2}"/>
     </joint>
     <link name="link_3">
@@ -165,5 +179,5 @@
            k_position="${safety_controller_k_pos}"
            k_velocity="${safety_controller_k_vel}"/>
-      <dynamics damping="${joint_damping}" friction="${joint_friction}"/>
+      <dynamics damping="${d3}" friction="${f3}"/>
     </joint>
     <link name="link_4">
@@ -200,5 +214,5 @@
            k_position="${safety_controller_k_pos}"
            k_velocity="${safety_controller_k_vel}"/>
-      <dynamics damping="${joint_damping}" friction="${joint_friction}"/>
+      <dynamics damping="${d4}" friction="${f4}"/>
     </joint>
     <link name="link_5">
@@ -235,5 +249,5 @@
            k_position="${safety_controller_k_pos}"
            k_velocity="${safety_controller_k_vel}"/>
-      <dynamics damping="${joint_damping}" friction="${joint_friction}"/>
+      <dynamics damping="${d5}" friction="${f5}"/>
     </joint>
     <link name="link_6">
@@ -270,5 +284,5 @@
            k_position="${safety_controller_k_pos}"
            k_velocity="${safety_controller_k_vel}"/>
-      <dynamics damping="${joint_damping}" friction="${joint_friction}"/>
+      <dynamics damping="${d6}" friction="${f6}"/>
     </joint>
     <link name="link_7">

File: urdf/iiwa14_ETHZ.xacro (robot description, xacro)
@@ -10,8 +10,22 @@
   <xacro:property name="safety_controller_k_pos" value="100" />
   <xacro:property name="safety_controller_k_vel" value="2" />
-  <xacro:property name="joint_damping" value="0.5" />
-  <xacro:property name="joint_friction" value="1.0" />
   <xacro:property name="max_effort" value="300"/>
   <xacro:property name="max_velocity" value="10"/>
+  <xacro:property name="damping_factor" value="1.0"/>
+   <xacro:property name="d0" value="${damping_factor*0.241499}"/>
+   <xacro:property name="d1" value="${damping_factor*0.373279}"/>
+   <xacro:property name="d2" value="${damping_factor*0.110253}"/>
+   <xacro:property name="d3" value="${damping_factor*0.100000}"/>
+   <xacro:property name="d4" value="${damping_factor*0.100000}"/>
+   <xacro:property name="d5" value="${damping_factor*0.124842}"/>
+   <xacro:property name="d6" value="${damping_factor*0.100000}"/>
+   <xacro:property name="friction_factor" value="1.0"/>
+   <xacro:property name="f0" value="${friction_factor*0.319088}"/>
+   <xacro:property name="f1" value="${friction_factor*0.181301}"/>
+   <xacro:property name="f2" value="${friction_factor*0.073019}"/>
+   <xacro:property name="f3" value="${friction_factor*0.176713}"/>
+   <xacro:property name="f4" value="${friction_factor*0.034631}"/>
+   <xacro:property name="f5" value="${friction_factor*0.133913}"/>
+   <xacro:property name="f6" value="${friction_factor*0.087096}"/>
   <xacro:macro name="iiwa14" params="parent hardware_interface robot_name *origin">
     <!--joint between {parent} and link_0-->
@@ -60,5 +74,5 @@
            k_position="${safety_controller_k_pos}"
            k_velocity="${safety_controller_k_vel}"/>
-      <dynamics damping="${joint_damping}" friction="${joint_friction}"/>
+      <dynamics damping="${d0}" friction="${f0}"/>
     </joint>
     <link name="link_1">
@@ -95,5 +109,5 @@
            k_position="${safety_controller_k_pos}"
            k_velocity="${safety_controller_k_vel}"/>
-      <dynamics damping="${joint_damping}" friction="${joint_friction}"/>
+      <dynamics damping="${d1}" friction="${f1}"/>
     </joint>
     <link name="link_2">
@@ -130,5 +144,5 @@
            k_position="${safety_controller_k_pos}"
            k_velocity="${safety_controller_k_vel}"/>
-      <dynamics damping="${joint_damping}" friction="${joint_friction}"/>
+      <dynamics damping="${d2}" friction="${f2}"/>
     </joint>
     <link name="link_3">
@@ -165,5 +179,5 @@
            k_position="${safety_controller_k_pos}"
            k_velocity="${safety_controller_k_vel}"/>
-      <dynamics damping="${joint_damping}" friction="${joint_friction}"/>
+      <dynamics damping="${d3}" friction="${f3}"/>
     </joint>
     <link name="link_4">
@@ -200,5 +214,5 @@
            k_position="${safety_controller_k_pos}"
            k_velocity="${safety_controller_k_vel}"/>
-      <dynamics damping="${joint_damping}" friction="${joint_friction}"/>
+      <dynamics damping="${d4}" friction="${f4}"/>
     </joint>
     <link name="link_5">
@@ -235,5 +249,5 @@
            k_position="${safety_controller_k_pos}"
            k_velocity="${safety_controller_k_vel}"/>
-      <dynamics damping="${joint_damping}" friction="${joint_friction}"/>
+      <dynamics damping="${d5}" friction="${f5}"/>
     </joint>
     <link name="link_6">
@@ -270,5 +284,5 @@
            k_position="${safety_controller_k_pos}"
            k_velocity="${safety_controller_k_vel}"/>
-      <dynamics damping="${joint_damping}" friction="${joint_friction}"/>
+      <dynamics damping="${d6}" friction="${f6}"/>
     </joint>
     <link name="link_7">

Commit message: Added MFT Pneumatisch flange

File: urdf/iiwa14.xacro (robot description, xacro)
@@ -12,5 +12,5 @@
   <xacro:property name="max_effort" value="300"/>
   <xacro:property name="max_velocity" value="10"/>
-   <xacro:property name="damping_factor" value="1.0"/>
+   <xacro:property name="damping_factor" value="0.0"/>
    <xacro:property name="d0" value="${damping_factor*0.1}"/>
    <xacro:property name="d1" value="${damping_factor*0.1}"/>
@@ -20,5 +20,5 @@
    <xacro:property name="d5" value="${damping_factor*0.1}"/>
    <xacro:property name="d6" value="${damping_factor*0.1}"/>
-   <xacro:property name="friction_factor" value="1.0"/>
+   <xacro:property name="friction_factor" value="0.0"/>
    <xacro:property name="f0" value="${friction_factor*0.1}"/>
    <xacro:property name="f1" value="${friction_factor*0.1}"/>
@@ -255,5 +255,5 @@
         <origin xyz="0 0.0006 0.0004" rpy="0 0 0"/>
         <mass value="1.8"/>
-        <inertia ixx="0.005"  ixy="0"  ixz="0" iyy="0.0036" iyz="0" izz="0.0047" />
+        <inertia ixx="0.025"  ixy="0"  ixz="0" iyy="0.0136" iyz="0" izz="0.0247" />
       </inertial>
       <visual>
@@ -289,11 +289,12 @@
       <inertial>
         <origin xyz="0 0 0.02" rpy="0 0 0"/>
-        <mass value="0.3"/>
-        <inertia ixx="0.001"  ixy="0"  ixz="0" iyy="0.001" iyz="0" izz="0.001" />
-      </inertial>
-      <visual>
-        <origin xyz="0 0 0" rpy="0 0 0"/>
-        <geometry>
-          <mesh filename="package://iiwa_description/meshes/iiwa14/visual/link_7.stl"/>
+        <mass value="${0.3 / 0.308 * 0.44}"/> <!--this is for the MFT Pneumatisch flange-->
+        <inertia ixx="0.01"  ixy="0"  ixz="0" iyy="0.01" iyz="0" izz="0.01" />
+      </inertial>
+      <visual>
+        <origin xyz="0 0 0" rpy="0 0 0"/>
+        <geometry>
+<!--           <mesh filename="package://iiwa_description/meshes/iiwa14/visual/link_7.stl"/> -->
+		  <mesh filename="package://iiwa_description/meshes/iiwa14/visual/link_7-MF-Touch-pneumatisch.stl"/>
         </geometry>
         <material name="Grey"/>
@@ -302,5 +303,6 @@
         <origin xyz="0 0 0" rpy="0 0 0"/>
         <geometry>
-          <mesh filename="package://iiwa_description/meshes/iiwa14/collision/link_7.stl"/>
+<!--           <mesh filename="package://iiwa_description/meshes/iiwa14/collision/link_7.stl"/> -->
+		  <mesh filename="package://iiwa_description/meshes/iiwa14/collision/link_7-MF-Touch-pneumatisch.stl"/>
         </geometry>
         <material name="Grey"/>
@@ -320,5 +322,12 @@
       <axis xyz="0 0 1"/>
     </joint>
+	<joint name="joint_ee_kuka_mft_pneum" type="fixed">
+      <parent link="link_7"/>
+      <child link="link_ee_kuka_mft_pneum"/>
+      <origin xyz="0 0 0.071" rpy="0 -${PI/2} 0"/>
+    </joint>
     <link name="link_ee_kuka">
+    </link>
+	<link name="link_ee_kuka_mft_pneum">
     </link>
     <!--Extensions -->

File: urdf/iiwa14_ETHZ.xacro (robot description, xacro)
@@ -12,5 +12,5 @@
   <xacro:property name="max_effort" value="300"/>
   <xacro:property name="max_velocity" value="10"/>
-  <xacro:property name="damping_factor" value="1.0"/>
+  <xacro:property name="damping_factor" value="0.0"/>
    <xacro:property name="d0" value="${damping_factor*0.241499}"/>
    <xacro:property name="d1" value="${damping_factor*0.373279}"/>
@@ -20,12 +20,12 @@
    <xacro:property name="d5" value="${damping_factor*0.124842}"/>
    <xacro:property name="d6" value="${damping_factor*0.100000}"/>
-   <xacro:property name="friction_factor" value="1.0"/>
-   <xacro:property name="f0" value="${friction_factor*0.319088}"/>
+   <xacro:property name="friction_factor" value="0.0"/>
+   <xacro:property name="f0" value="${friction_factor*0.319088	*	1.0 }"/>
    <xacro:property name="f1" value="${friction_factor*0.181301}"/>
    <xacro:property name="f2" value="${friction_factor*0.073019}"/>
    <xacro:property name="f3" value="${friction_factor*0.176713}"/>
-   <xacro:property name="f4" value="${friction_factor*0.034631}"/>
+   <xacro:property name="f4" value="${friction_factor*0.034631	*	1.0 }"/>
    <xacro:property name="f5" value="${friction_factor*0.133913}"/>
-   <xacro:property name="f6" value="${friction_factor*0.087096}"/>
+   <xacro:property name="f6" value="${friction_factor*0.087096 	*	1.0 }"/>
   <xacro:macro name="iiwa14" params="parent hardware_interface robot_name *origin">
     <!--joint between {parent} and link_0-->
@@ -289,5 +289,5 @@
       <inertial>
         <origin xyz="-0.03465 -0.023242 ${0.071377-0.081}" rpy="0 0 0"/>
-        <mass value="0.354321"/>
+        <mass value="${0.354321 / 0.308 * 0.44}"/> <!--this is for the MFT Pneumatisch flange-->
         <inertia ixx="0.007946"  ixy="0.000221"  ixz="0.000294" iyy="0.010889" iyz="-0.000294" izz="0.002944" />
       </inertial>

Commit message: simplified meshes - ok - so long suckers

File: urdf/iiwa14.xacro (robot description, xacro)
@@ -51,5 +51,5 @@
         <origin xyz="0 0 0" rpy="0 0 0"/>
         <geometry>
-          <mesh filename="package://iiwa_description/meshes/iiwa14/collision/link_0.stl"/>
+          <mesh filename="package://iiwa_description/meshes/iiwa14/collision/link_0_s.stl"/>
         </geometry>
         <material name="Grey"/>
@@ -92,5 +92,5 @@
         <origin xyz="0 0 0" rpy="0 0 0"/>
         <geometry>
-          <mesh filename="package://iiwa_description/meshes/iiwa14/collision/link_1.stl"/>
+          <mesh filename="package://iiwa_description/meshes/iiwa14/collision/link_1_s.stl"/>
         </geometry>
         <material name="Orange"/>
@@ -127,5 +127,5 @@
         <origin xyz="0 0 0" rpy="0 0 0"/>
         <geometry>
-          <mesh filename="package://iiwa_description/meshes/iiwa14/collision/link_2.stl"/>
+          <mesh filename="package://iiwa_description/meshes/iiwa14/collision/link_2_s.stl"/>
         </geometry>
         <material name="Orange"/>
@@ -162,5 +162,5 @@
         <origin xyz="0 0 0" rpy="0 0 0"/>
         <geometry>
-          <mesh filename="package://iiwa_description/meshes/iiwa14/collision/link_3.stl"/>
+          <mesh filename="package://iiwa_description/meshes/iiwa14/collision/link_3_s.stl"/>
         </geometry>
         <material name="Orange"/>
@@ -197,5 +197,5 @@
         <origin xyz="0 0 0" rpy="0 0 0"/>
         <geometry>
-          <mesh filename="package://iiwa_description/meshes/iiwa14/collision/link_4.stl"/>
+          <mesh filename="package://iiwa_description/meshes/iiwa14/collision/link_4_s.stl"/>
         </geometry>
         <material name="Orange"/>
@@ -232,5 +232,5 @@
         <origin xyz="0 0 0" rpy="0 0 0"/>
         <geometry>
-          <mesh filename="package://iiwa_description/meshes/iiwa14/collision/link_5.stl"/>
+          <mesh filename="package://iiwa_description/meshes/iiwa14/collision/link_5_s.stl"/>
         </geometry>
         <material name="Orange"/>
@@ -267,5 +267,5 @@
         <origin xyz="0 0 0" rpy="0 0 0"/>
         <geometry>
-          <mesh filename="package://iiwa_description/meshes/iiwa14/collision/link_6.stl"/>
+          <mesh filename="package://iiwa_description/meshes/iiwa14/collision/link_6_s.stl"/>
         </geometry>
         <material name="Orange"/>
@@ -303,6 +303,6 @@
         <origin xyz="0 0 0" rpy="0 0 0"/>
         <geometry>
-<!--           <mesh filename="package://iiwa_description/meshes/iiwa14/collision/link_7.stl"/> -->
-		  <mesh filename="package://iiwa_description/meshes/iiwa14/collision/link_7-MF-Touch-pneumatisch.stl"/>
+<!--           <mesh filename="package://iiwa_description/meshes/iiwa14/collision/link_7_s.stl"/> -->
+		  <mesh filename="package://iiwa_description/meshes/iiwa14/collision/link_7-MF-Touch-pneumatisch_s.stl"/>
         </geometry>
         <material name="Grey"/>
