Commit message: update joint names

File: urdf/iiwa.gazebo.xacro (robot description, xacro)
@@ -1,28 +1,13 @@
 <?xml version="1.0"?>
 <robot xmlns:xacro="http://www.ros.org/wiki/xacro">
-    <xacro:arg name="load_gazebo_ros_control" default="false"/>
-    <xacro:macro  name="gz_joint" params="joint_name">
-        <gazebo reference="${joint_name}">
-            <provideFeedback>true</provideFeedback>
-        </gazebo>
-    </xacro:macro>
-    <xacro:gz_joint joint_name="joint_0"/>
-    <xacro:gz_joint joint_name="joint_1"/>
-    <xacro:gz_joint joint_name="joint_2"/>
-    <xacro:gz_joint joint_name="joint_3"/>
-    <xacro:gz_joint joint_name="joint_4"/>
-    <xacro:gz_joint joint_name="joint_5"/>
-    <xacro:gz_joint joint_name="joint_6"/>
   <xacro:macro name="iiwa_gazebo" params="robot_name">
     <!-- Load Gazebo lib and set the robot namespace -->
-    <gazebo>
-        <xacro:if value="$(arg load_gazebo_ros_control)">
-          <plugin name="gazebo_ros_control" filename="libgazebo_ros_control.so">
-            <!--robotNamespace>/${robot_name}</robotNamespace-->
-          </plugin>
-        </xacro:if>
-    </gazebo>
+    <!-- <gazebo>
+      <plugin name="gazebo_ros_control" filename="libgazebo_ros_control.so">
+        <robotNamespace>/${robot_name}</robotNamespace>
+      </plugin>
+    </gazebo> -->
     <!-- Link0 -->
-    <gazebo reference="link_0">
+    <gazebo reference="${robot_name}_link_0">
       <material>Gazebo/Grey</material>
       <mu1>0.2</mu1>
@@ -30,5 +15,5 @@
     </gazebo>
     <!-- Link1 -->
-    <gazebo reference="link_1">
+    <gazebo reference="${robot_name}_link_1">
       <material>Gazebo/Orange</material>
       <mu1>0.2</mu1>
@@ -36,5 +21,5 @@
     </gazebo>
     <!-- Link2 -->
-    <gazebo reference="link_2">
+    <gazebo reference="${robot_name}_link_2">
       <material>Gazebo/Orange</material>
       <mu1>0.2</mu1>
@@ -42,5 +27,5 @@
     </gazebo>
     <!-- Link3 -->
-    <gazebo reference="link_3">
+    <gazebo reference="${robot_name}_link_3">
       <material>Gazebo/Orange</material>
       <mu1>0.2</mu1>
@@ -48,5 +33,5 @@
     </gazebo>
     <!-- Link4 -->
-    <gazebo reference="link_4">
+    <gazebo reference="${robot_name}_link_4">
       <material>Gazebo/Orange</material>
       <mu1>0.2</mu1>
@@ -54,5 +39,5 @@
     </gazebo>
     <!-- Link5 -->
-    <gazebo reference="link_5">
+    <gazebo reference="${robot_name}_link_5">
       <material>Gazebo/Orange</material>
       <mu1>0.2</mu1>
@@ -60,5 +45,5 @@
     </gazebo>
     <!-- Link6 -->
-    <gazebo reference="link_6">
+    <gazebo reference="${robot_name}_link_6">
       <material>Gazebo/Orange</material>
       <mu1>0.2</mu1>
@@ -66,5 +51,5 @@
     </gazebo>
     <!-- Link7 -->
-    <gazebo reference="link_7">
+    <gazebo reference="${robot_name}_link_7">
       <material>Gazebo/Grey</material>
       <mu1>0.2</mu1>

File: urdf/iiwa.transmission.xacro (robot description, xacro)
@@ -2,70 +2,77 @@
 <robot xmlns:xacro="http://www.ros.org/wiki/xacro">
   <xacro:macro name="iiwa_transmission" params="hardware_interface">
-    <transmission name="iiwa_tran_0">
+    <transmission name="${robot_name}_tran_1">
+      <robotNamespace>/${robot_name}</robotNamespace>
       <type>transmission_interface/SimpleTransmission</type>
-      <joint name="joint_0">
+      <joint name="${robot_name}_joint_1">
 	<hardwareInterface>${hardware_interface}</hardwareInterface>
       </joint>
-      <actuator name="iiwa_motor_0">
+      <actuator name="${robot_name}_motor_1">
 	<hardwareInterface>${hardware_interface}</hardwareInterface>
 	<mechanicalReduction>1</mechanicalReduction>
       </actuator>
     </transmission>
-    <transmission name="iiwa_tran_1">
+    <transmission name="${robot_name}_tran_2">
+      <robotNamespace>/${robot_name}</robotNamespace>
       <type>transmission_interface/SimpleTransmission</type>
-      <joint name="joint_1">
+      <joint name="${robot_name}_joint_2">
 	<hardwareInterface>${hardware_interface}</hardwareInterface>
       </joint>
-      <actuator name="iiwa_motor_1">
+      <actuator name="${robot_name}_motor_2">
 	<hardwareInterface>${hardware_interface}</hardwareInterface>
 	<mechanicalReduction>1</mechanicalReduction>
       </actuator>
     </transmission>
-    <transmission name="iiwa_tran_2">
+    <transmission name="${robot_name}_tran_3">
+      <robotNamespace>/${robot_name}</robotNamespace>
       <type>transmission_interface/SimpleTransmission</type>
-      <joint name="joint_2">
+      <joint name="${robot_name}_joint_3">
 	<hardwareInterface>${hardware_interface}</hardwareInterface>
       </joint>
-      <actuator name="iiwa_motor_2">
+      <actuator name="${robot_name}_motor_3">
 	<hardwareInterface>${hardware_interface}</hardwareInterface>
 	<mechanicalReduction>1</mechanicalReduction>
       </actuator>
     </transmission>
-    <transmission name="iiwa_tran_3">
+    <transmission name="${robot_name}_tran_4">
+      <robotNamespace>/${robot_name}</robotNamespace>
       <type>transmission_interface/SimpleTransmission</type>
-      <joint name="joint_3">
+      <joint name="${robot_name}_joint_4">
 	<hardwareInterface>${hardware_interface}</hardwareInterface>
       </joint>
-      <actuator name="iiwa_motor_3">
+      <actuator name="${robot_name}_motor_4">
 	<hardwareInterface>${hardware_interface}</hardwareInterface>
 	<mechanicalReduction>1</mechanicalReduction>
       </actuator>
     </transmission>
-    <transmission name="iiwa_tran_4">
+    <transmission name="${robot_name}_tran_5">
+      <robotNamespace>/${robot_name}</robotNamespace>
       <type>transmission_interface/SimpleTransmission</type>
-      <joint name="joint_4">
+      <joint name="${robot_name}_joint_5">
 	<hardwareInterface>${hardware_interface}</hardwareInterface>
       </joint>
-      <actuator name="iiwa_motor_4">
+      <actuator name="${robot_name}_motor_5">
 	<hardwareInterface>${hardware_interface}</hardwareInterface>
 	<mechanicalReduction>1</mechanicalReduction>
       </actuator>
     </transmission>
-    <transmission name="iiwa_tran_5">
+    <transmission name="${robot_name}_tran_6">
+      <robotNamespace>/${robot_name}</robotNamespace>
       <type>transmission_interface/SimpleTransmission</type>
-      <joint name="joint_5">
+      <joint name="${robot_name}_joint_6">
 	<hardwareInterface>${hardware_interface}</hardwareInterface>
       </joint>
-      <actuator name="iiwa_motor_5">
+      <actuator name="${robot_name}_motor_6">
 	<hardwareInterface>${hardware_interface}</hardwareInterface>
 	<mechanicalReduction>1</mechanicalReduction>
       </actuator>
     </transmission>
-    <transmission name="iiwa_tran_6">
+    <transmission name="${robot_name}_tran_7">
+      <robotNamespace>/${robot_name}</robotNamespace>
       <type>transmission_interface/SimpleTransmission</type>
-      <joint name="joint_6">
+      <joint name="${robot_name}_joint_7">
 	<hardwareInterface>${hardware_interface}</hardwareInterface>
       </joint>
-      <actuator name="iiwa_motor_6">
+      <actuator name="${robot_name}_motor_7">
 	<hardwareInterface>${hardware_interface}</hardwareInterface>
 	<mechanicalReduction>1</mechanicalReduction>
